File: PCB/Battery Charger/Battery Charger.sch (KiCad schematic (older format))
At the start: 28 parts

Commit message: code works, but modified control law so that its based on error in the signal.  try a small pertubation, a good looking one is q1 = -3.137 q2 = 0.04.
Parts:
- removed BT?: BATTERY, ~, symbol BATTERY
- added K?: PIC, symbol CONN_3
- added P?: WALL, symbol CONN_2
- added P?: SYS, symbol CONN_2
- added P?: BAT, symbol CONN_2
- TH?: value THERMISTOR -> NTC_THERMISTOR
Connections:
- net GND: now also R?.1, U?.4 (GND), P?.2 (PM), P?.2 (PM), P?.2 (PM)
- net VIN: now reaches R?.1, R?.2, U?.27 (IN)
- net VIN: now also P?.1 (P1)
- net at U?.11 (~FLT): now also K?.2 (PM)
- net at U?.12 (~CHRG): now also K?.3 (P3)
- net VBAT: now reaches Q?.D, R?.2, U?.17 (BAT)
- net VBAT: now also P?.1 (P1)
- net VSYS: now reaches Q?.S, R?.1, R?.2, U?.20 (CSP)
- net VSYS: now also P?.1 (P1)
- net at U?.5 (ENC): now also K?.1 (P1)
Other:
- note added: "For current limited by RIS and RCS sense resistors leave CL and IL disconnected.\n\nThe battery manager chips give similar information outputted by IIMON and IBMON.\nAdding capacitors to IIMON and IBMON could affet internal control loops so it is\ndisconnected for now."
