File: PCB/Battery Parts Test PCB/2_power.sch (KiCad schematic (older format))
At the start: 6 parts, among them K2 CONN_3, U2 ATA6870

Commit message: updated schematic
Changed lines of the file:
@@
-EESchema Schematic File Version 2  date 4/30/2013 1:48:29 PM
+EESchema Schematic File Version 2  date 5/7/2013 3:13:49 PM
 LIBS:power
 LIBS:device
@@
 Sheet 7 9
 Title ""
-Date "30 apr 2013"
+Date "7 may 2013"
 Rev ""
 Comp ""
@@
 Connection ~ 4800 2850
 Wire Wire Line
-	3550 2850 3550 4550
+	3550 4550 3550 2850
 Wire Wire Line
-	5300 2850 3550 2850
+	3550 2850 5300 2850
 Connection ~ 6900 3200
 Wire Wire Line
@@
 	5300 3450 5150 3450
 Wire Wire Line
-	6900 3100 6800 3100
+	6800 3100 6900 3100
 Wire Wire Line
-	6900 4050 6900 3100
+	6900 3100 6900 4050
 Connection ~ 6900 4050
 Wire Wire Line
@@
 Connection ~ 6900 3300
 Wire Wire Line
-	3650 3500 3250 3500
+	3250 3500 3650 3500
 Wire Wire Line
-	3650 4550 3650 3500
+	3650 3500 3650 4550
 Wire Wire Line
-	3750 4050 7650 4050
+	7650 4050 3750 4050
 Wire Wire Line
-	3750 4550 3750 4050
+	3750 4050 3750 4550
 Connection ~ 4200 4050
 Wire Wire Line
