File: PCB/Battery Parts Test PCB/battery_manager.sch (KiCad schematic (older format))
At the start: 10 parts

Commit message: updated schematic
Parts:
- gave numbers to parts that had none: 10
Connections:
- net PD_N: now reaches TP3.1, U1.38 (PD_N)
