File: PCB/Battery Parts Test PCB/misc_io.sch (KiCad schematic (older format))
At the start: 9 parts, among them P2 CONN_4X2, P3 CONN_13X2

Commit message: finished schematic with new battery monitor
Parts:
- removed C12, C13: 0.1uF, symbol C
- removed P2: CONN_4X2, symbol CONN_4X2
- removed P3: CONN_13X2, symbol CONN_13X2
- removed R41, R42, R43, R44, R45: 10K, symbol R
Connections:
- no-connect marks 23 -> 0
Other:
- note removed: "PSD might be best setting up an LED\n"

Commit message: updated schematic
Parts:
- added P2: CONN_5X2, symbol CONN_5X2
- added R58, R59: 1K, symbol R
Connections:
- new net +3.3V: P2.1, R58.1, R59.1
- new net CLK: P2.8
- new net CS_N: P2.6
- new net DGND: P2.9
- new net IRQ: P2.10, R59.2
- new net MISO: P2.5, R58.2
- new net MOSI: P2.4
- new net SCK: P2.3
- no-connect marks 0 -> 2
Changed lines of the file:
@@
-EESchema Schematic File Version 2  date 4/30/2013 1:48:29 PM
+EESchema Schematic File Version 2  date 5/7/2013 3:13:49 PM
 LIBS:power
 LIBS:device
@@
 Sheet 4 9
 Title ""
-Date "30 apr 2013"
+Date "7 may 2013"
 Rev ""
 Comp ""
@@
 Comment4 ""
 $EndDescr
+Connection ~ 4050 2850
+Wire Wire Line
+	5550 3050 5100 3050
+Wire Wire Line
+	5550 2950 5100 2950
+Wire Wire Line
+	3850 2750 4300 2750
+Wire Wire Line
+	5550 2750 5100 2750
+Wire Wire Line
+	3850 2850 4300 2850
+Wire Wire Line
+	5550 2850 5100 2850
+Connection ~ 5400 3050
+$Comp
+L R R58
+U 1 1 5184844A
+P 4050 2600
+F 0 "R58" V 4130 2600 50  0000 C CNN
+F 1 "1K" V 4050 2600 50  0000 C CNN
+	1    4050 2600
+	1    0    0    -1
+$EndComp
+$Comp
+L +3.3V #PWR06
+U 1 1 51848449
+P 4050 2350
+F 0 "#PWR06" H 4050 2310 30  0001 C CNN
+F 1 "+3.3V" H 4050 2460 30  0000 C CNN
+	1    4050 2350
+	1    0    0    -1
+$EndComp
+$Comp
+L +3.3V #PWR07
+U 1 1 51848433
+P 5400 2550
+F 0 "#PWR07" H 5400 2510 30  0001 C CNN
+F 1 "+3.3V" H 5400 2660 30  0000 C CNN
+	1    5400 2550
+	1    0    0    -1
+$EndComp
+NoConn ~ 5100 2650
+$Comp
+L +3.3V #PWR08
+U 1 1 51848334
+P 4300 2650
+F 0 "#PWR08" H 4300 2610 30  0001 C CNN
+F 1 "+3.3V" H 4300 2760 30  0000 C CNN
+	1    4300 2650
+	1    0    0    -1
+$EndComp
+$Comp
+L DGND #PWR09
+U 1 1 5184832A
+P 4300 3050
+F 0 "#PWR09" H 4300 3050 40  0001 C CNN
+F 1 "DGND" H 4300 2980 40  0000 C CNN
+	1    4300 3050
+	1    0    0    -1
+$EndComp
+NoConn ~ 4300 2950
+$Comp
+L R R59
+U 1 1 51848113
+P 5400 2800
+F 0 "R59" V 5480 2800 50  0000 C CNN
+F 1 "1K" V 5400 2800 50  0000 C CNN
+	1    5400 2800
+	1    0    0    -1
+$EndComp
+$Comp
+L CONN_5X2 P2
+U 1 1 51847E55
+P 4700 2850
+F 0 "P2" H 4700 3150 60  0000 C CNN
+F 1 "CONN_5X2" V 4700 2850 50  0000 C CNN
+	1    4700 2850
+	1    0    0    -1
+$EndComp
+Text HLabel 5550 2850 2    60   Input ~ 0
+CS_N
+Text HLabel 5550 2950 2    60   Input ~ 0
+CLK
+Text HLabel 3850 2750 0    60   Input ~ 0
+SCK
+Text HLabel 3850 2850 0    60   Input ~ 0
+MISO
+Text HLabel 5550 2750 2    60   Input ~ 0
+MOSI
+Text HLabel 5550 3050 2    60   Input ~ 0
+IRQ
 $EndSCHEMATC
