File: PCB/Motor & Magnet PCB/MotorMagnet PCB.sch (KiCad schematic (older format))
At the start: 19 parts

Commit message: Updated Motor/Magnet PCB
Parts:
- added C15, C16, C17: 1nF, ~, symbol C
- added C18, C19, C20, C21, C22, C23: DNI, ~, symbol C
- added C45, C46, C47: 0.1nF, ~, symbol C
- added K1, K2: CONN_3, symbol CONN_3
- added R10, R5, R6, R7, R8, R9: DNI, ~, symbol R
- added R11, R12, R13: 330, ~, symbol R
Connections:
- net labels added: MotorOut0, MotorOut1, MotorOut2
- wire segments 73 -> 173
Other:
- note added: "3 Phase Motor Connector"
- note added: "Jumper to set all chips to have FAULT_EN protection"
- note added: "MotorOut[0..2]"
- moved on the sheet: C2, C5, Current Sensor, D?, LED, P?, R, R1, R?, XBEE Chip
