File: PCB/Motor & Magnet PCB/_autosave-MotorMagnet.kicad_pcb (KiCad board)
At the start: 2 copper layers, 0 parts

Commit message: Motor/Magnet updates
(from earlier in the week)
Parts:
- added C15: 1nF, C1, F.Cu at (238.8, 88.9)
- added C16: 1nF, C1, F.Cu at (264.2, 68.6)
- added C17: 1nF, C1, F.Cu at (265.4, 87.6)
- added C18: DNI, C1, F.Cu at (276.9, 86.4)
- added C19: DNI, C1, F.Cu at (214.6, 63.5)
- added C2: 10uF, C1, F.Cu at (177.2, 100.3)
- added C20: DNI, C1, F.Cu at (281.9, 76.2)
- added C21: DNI, C1, F.Cu at (86.4, 44.5)
- added C22: DNI, C1, F.Cu at (205.7, 49.5)
- added C23: DNI, C1, F.Cu at (259.1, 55.9)
- added C45: 0.1nF, C1, F.Cu at (268.0, 49.5)
- added C46: 0.1nF, C1, F.Cu at (226.7, 113.0)
- added C47: 0.1nF, C1, F.Cu at (85.1, 53.3)
- added C5: 0.1uF, C1, F.Cu at (135.9, 108.6)
- added Current1: ACS716, DIP-16__300, F.Cu at (262.9, 77.5)
- added Current2: ACS716, DIP-16__300, F.Cu at (226.1, 80.0)
- added Current3: ACS716, DIP-16__300, F.Cu at (142.2, 159.4)
- added D1: ZENER 24V, D3, F.Cu at (139.7, 54.6)
- added D2: ZENER 3.3V, D3, F.Cu at (129.5, 27.9)
- added D3: ZENER 5V, D3, F.Cu at (108.0, 58.4)
- added J1: BREADBOARD_HEADER_L, pin_array_13x2, F.Cu at (147.3, 96.5)
- added J2: JP5, PIN_ARRAY_5x1, F.Cu at (142.2, 106.7)
- added J3: BREADBOARD_HEADER_R, pin_array_13x2, F.Cu at (172.7, 105.4)
- added K1: CONN_3, PIN_ARRAY_3X1, F.Cu at (231.1, 40.6)
- added K2: CONN_3, PIN_ARRAY_3X1, F.Cu at (243.8, 69.8)
- added LED1: D, LED-5MM, F.Cu at (151.1, 145.4)
- added P1: CONN_6, PIN_ARRAY-6X1, F.Cu at (208.3, 71.1)
- added R1: 2.2k, R1, F.Cu at (137.8, 102.9)
- added R10: DNI, R1, F.Cu at (238.8, 95.2)
- added R11: 330, R1, F.Cu at (223.5, 53.3)
- added R12: 330, R1, F.Cu at (219.7, 91.4)
- added R13: 330, R1, F.Cu at (271.8, 94.0)
- added R14: 2.2K, R1, F.Cu at (246.4, 83.8)
- added R15: 2.2K, R1, F.Cu at (236.2, 55.9)
- added R16: 2.2K, R1, F.Cu at (260.4, 49.5)
- added R17: R, R1, F.Cu at (156.2, 138.4)
- added R2: R, R1, F.Cu at (241.3, 54.6)
- added R3: R, R1, F.Cu at (227.3, 50.8)
- added R4: 168.3, R1, F.Cu at (222.2, 68.6)
- added R5: DNI, R1, F.Cu at (118.1, 53.3)
- added R6: DNI, R1, F.Cu at (127.0, 63.5)
- added R7: DNI, R1, F.Cu at (210.8, 90.2)
- added R8: DNI, R1, F.Cu at (248.9, 94.0)
- added R9: DNI, R1, F.Cu at (261.6, 94.0)
- added U$11: DSPIC33FJ12MC202, DIP-28__600, F.Cu at (160.0, 101.6)
- added XBEE1: XBEE-1B2, DIP-20__300, F.Cu at (152.4, 130.2)
Routing:
- net /PVDD: track 0.00 -> 30.9 mm
- net /PVSS: track 0.00 -> 30.1 mm
- net /PMCLR: track 0.00 -> 27.4 mm
- net N-0000017: track 0.00 -> 14.7 mm
- net N-0000016: track 0.00 -> 14.7 mm
- net N-000005: track 0.00 -> 12.6 mm
- net /PVCAP: track 0.00 -> 12.5 mm
- net /PGD: track 0.00 -> 10.7 mm
- net /PGC: track 0.00 -> 10.7 mm
- net N-0000010: track 0.00 -> 9.09 mm
- net N-000007: track 0.00 -> 3.81 mm
- net N-0000067: track 0.00 -> 3.81 mm
- net N-0000066: track 0.00 -> 3.81 mm
- net N-0000065: track 0.00 -> 3.81 mm
- net N-0000061: track 0.00 -> 3.81 mm
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