File: PCB/New PCB/sensors.sch (KiCad schematic (older format))
At the start: 24 parts

Commit message: Updating Schematic for New PCB
Parts:
- added ACCELEROMETER2: AIS328DQ, ~, symbol AIS328DQ
- added C11, C24, C28, C29, C3, C33: 0.1 uF, ~, symbol C
- added C13, C14, C31, C32: C, ~, symbol C
- added C15, C16: C1 nF, ~, symbol C
- added C18, C19, C21, C22: DNI, ~, symbol C
- added C25, C26: 1uF, ~, symbol C
- added C6: 10 nF, ~, symbol C
- added C7: 470 nF, ~, symbol C
- added CURRENT1, CURRENT2: ACS716, symbol ACS716
- added GYROSCOPE2: A3G4250D, ~, symbol A3G4250D
- added JP2, JP3: JP, symbol JP
- added JP5, JP6: MOT_ENC, symbol MOT_ENC
- added MAGNET2, MOTOR1: LS7366RDIP, symbol LS7366RDIP
- added R11, R12: 330, ~, symbol R
- added R14, R4: R, ~, symbol R
- added R2: 10K, ~, symbol R
- added R5, R6, R7, R8: DNI, ~, symbol R
- added X2, X3: 20 MHz, ~, symbol QUARTZCMS4
- gave numbers to parts that had none: 24
Connections:
- net labels added: ANC1, ANC2, ANC3, DIO3, DIO4, DIO5, DIO6, DIO7
- net labels removed: SPI_SS
- wire segments 134 -> 356
Other:
- moved on the sheet: C17, C20, C23, C27, C30, CURRENT3, R10, R13, R9

Commit message: updated schematic
Parts:
- removed C10, C11, C12, C2, C24, C3: 0.1 uF, ~, symbol C
- removed C13, C14, C8, C9: C, ~, symbol C
- removed JP1, JP5: MOT_ENC, symbol MOT_ENC
- removed JP2, JP3, JP4: JP, symbol JP
- removed MAGNET1, MAGNET2: LS7366RDIP, symbol LS7366RDIP
- removed R3, R4: R, ~, symbol R
- removed X1, X2: 20 MHz, ~, symbol QUARTZCMS4
- added C? (x11): 0.1uF, symbol C
Connections:
- net labels removed: DIO5, DIO6
- wire segments 356 -> 250
Other:
- moved on the sheet: C15, C16, C17, C18, C19, C20, C21, C22, C23, C25, C26, C27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

Commit message: more updates
Other:
- moved on the sheet: ACCELEROMETER1, ACCELEROMETER2, C15, C16, C17, C18, C19, C20, C21, C22, C23, C25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

Commit message: updated schematic
Parts:
- removed ACCELEROMETER2: AIS328DQ, ~, symbol AIS328DQ
- removed C6: 10 nF, ~, symbol C
- removed C7: 470 nF, ~, symbol C
- removed C? (x4): 0.1uF, symbol C
- removed GYROSCOPE2: A3G4250D, ~, symbol A3G4250D
- removed R2: 10K, ~, symbol R
- added K1, K2: CONN_3, symbol CONN_3
- R14: value R -> 1M
- gave numbers to parts that had none: 7
Connections:
- net labels added: ACCEL1, ACCEL2, ACCEL3, ACCEL[1:3], ENC1, ENC2, ENC3, ENC[1:3], GYRO1, GYRO2, GYRO3, GYRO[1:3], MotorOut0, MotorOut1, MotorOut2, MotorOut[0:2], SPI_BUS[1:3]
- net labels removed: DFLAG, DIO1, DIO2, DIO3, DIO4, DIO7, INT1, INT2, INT_1, INT_2, LFLAG
- wire segments 250 -> 195
Other:
- note added: "3 Phase Motor Connector"
- note added: "Accelerometer, Gyro, Opposite Link QEI"
- note added: "Jumper to set all chips to have FAULT_EN protection"
- note added: "Motor Current Sensing"
- moved on the sheet: C33

Commit message: updated schematic and netlist, added flyback diodes
Parts:
- removed C28, C29, C30: 0.1 uF, ~, symbol C
- C15, C16, C17: value C1 nF -> 1nF
- C31, C32: value C -> 0.1uF
Connections:
- net ACCEL3 is gone; now on net ACCEL2: ACCELEROMETER1.7 (INT_1)
- net ENC3 is gone; now on net ENC2: MOTOR1.9 (~DFLAG)
- net GYRO3 is gone; now on net GYRO2: GYROSCOPE1.6 (DRDY/INT2)
- net ACCEL1: now also ACCELEROMETER1.3 (INT_2); no longer ACCELEROMETER1.12 (CS)
- net ACCEL2: no longer ACCELEROMETER1.3 (INT_2)
- net ANC1: now also CURRENT2.12 (VIOUT); no longer CURRENT3.12 (VIOUT)
- net ANC2: now also CURRENT3.12 (VIOUT); no longer CURRENT2.12 (VIOUT)
- net ENC1: now also MOTOR1.8 (~LFLAG); no longer MOTOR1.4 (~SS)
- net ENC2: no longer MOTOR1.8 (~LFLAG)
- net GYRO1: now also GYROSCOPE1.7 (INT1); no longer GYROSCOPE1.5 (CS)
- net GYRO2: no longer GYROSCOPE1.7 (INT1)
- net ANC3 renamed ANC0
- net SPI_CLK renamed SPI_BUS0
- net SPI_DIN renamed SPI_BUS1
- net SPI_DOUT renamed SPI_BUS2
- new net ACCEL0: ACCELEROMETER1.12 (CS)
- new net ENC0: MOTOR1.4 (~SS)
- new net GYRO0: GYROSCOPE1.5 (CS)
Other:
- note added: "SPI_BUS0 - CLK\nSPI_BUS1 - DIN\nSPI_BUS2 - DOUT"

Commit message: order has been placed and confirmed, receipt in project folder
Parts:
- removed C25, C26, C27: 1uF, ~, symbol C
- removed CURRENT1, CURRENT2, CURRENT3: ACS716, symbol ACS716
- added U7, U8, U9: ACS716, ~, symbol ACS716
- C33: value 0.1 uF -> 0.1uF
Connections:
- net ANC0: now also U7.12 (VIOUT)
- net ANC1: now also U8.12 (VIOUT)
- net ANC2: now also U9.12 (VIOUT)
- net GND: now also U7.9 (GND), U8.9 (GND), U9.9 (GND)
- net MotorOut0: now also U7.1 (IP+), U7.2 (IP+), U7.3 (IP+), U7.4 (IP+)
- net MotorOut1: now also U8.1 (IP+), U8.2 (IP+), U8.3 (IP+), U8.4 (IP+)
- net MotorOut2: now also U9.1 (IP+), U9.2 (IP+), U9.3 (IP+), U9.4 (IP+)
- net VCC: now also U7.14 (VCC), U8.14 (VCC), U9.14 (VCC)
- net at C17.1: now also U9.10 (VZCR)
- net at C20.1: now also U9.11 (FILTER)
- net at C23.1, R13.1: now also U9.13 (~FAULT)
- net at R10.1, R9.1: now also U9.15 (VOC)
- net at K2.2 (PM): now also U7.16 (FAULT_EN), U8.16 (FAULT_EN), U9.16 (FAULT_EN)
- net at K1.3 (P3): now also U9.5 (IP-), U9.6 (IP-), U9.7 (IP-), U9.8 (IP-)
- net at C22.1, R12.1: now also U8.13 (~FAULT)
- net at C19.1: now also U8.11 (FILTER)
- net at C16.1: now also U8.10 (VZCR)
- net at R7.1, R8.1: now also U8.15 (VOC)
- net at K1.2 (PM): now also U8.5 (IP-), U8.6 (IP-), U8.7 (IP-), U8.8 (IP-)
- net at C21.1, R11.1: now also U7.13 (~FAULT)
- net at C18.1: now also U7.11 (FILTER)
- net at C15.1: now also U7.10 (VZCR)
- net at R5.1, R6.1: now also U7.15 (VOC)
- net at K1.1 (P1): now also U7.5 (IP-), U7.6 (IP-), U7.7 (IP-), U7.8 (IP-)
