File: PCB/New PCB/power.sch (KiCad schematic (older format))
At the start: 49 parts, among them P1 BATT_CONN, P20 CONN_1, P21 CONN_1, P22 CONN_1, P23 CONN_1, P24 CONN_1, SW1 SPST, U1 DSPIC33EP512MC806, U2 1074HV, U3 1074HV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

Commit message: Fixes to Schematics
Parts:
- removed U1: DSPIC33EP512MC806, ~, symbol DSPIC33EP512MC806
Changed lines of the file:
@@
 Sheet 2 4
 Title ""
-Date "8 jul 2013"
+Date "15 jul 2013"
 Rev ""
 Comp ""
@@
 	0    -1   -1   0
 $EndComp
-$Comp
-L DSPIC33EP512MC806 U1
-U 2 1 51A3CE47
-P 9000 1200
-F 0 "U1" H 9000 1650 60  0000 C CNN
-F 1 "DSPIC33EP512MC806" H 9050 1550 60  0000 C CNN
-F 2 "~" H 9000 1200 60  0000 C CNN
-F 3 "~" H 9000 1200 60  0000 C CNN
-	2    9000 1200
-	1    0    0    -1
-$EndComp
 Text Notes 3950 700  0    60   ~ 0
