File: PCB/DsPIC Breakout/DsPIC Breakout.kicad_pcb (KiCad board)
At the start: 2 copper layers, 34.5 x 81.5 mm, 14 parts, among them J1 BREADBOARD_HEADER_32X1, J2 BREADBOARD_HEADER_32X1, P1 CONN_2, P2 PROG_H, U1 DSPIC33EP512MC806

Commit message: BreakoutBoard dsPIC64 PCB
Including final gerber files
Routing:
- net N-0000050: track 55.5 -> 44.7 mm
- net N-0000031: track 47.6 -> 37.3 mm
- net VCC: track 208.0 -> 198.3 mm
- net N-0000027: track 46.5 -> 37.2 mm
- net N-0000049: track 48.6 -> 39.5 mm
- net N-0000029: track 51.6 -> 42.6 mm
- net N-0000036: track 47.8 -> 39.1 mm
- net N-0000028: track 40.4 -> 32.0 mm
- net N-0000048: track 43.0 -> 34.7 mm
- net N-0000030: track 37.5 -> 29.7 mm
- net N-0000037: track 40.7 -> 34.5 mm
- net N-000008: track 106.8 -> 101.0 mm
- net N-0000032: track 38.3 -> 32.9 mm
- net N-0000035: track 47.0 -> 41.8 mm
- net N-0000051: track 27.9 -> 24.3 mm
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Other:
- board text added: "1) PWM3H (MotorCon5)"
- board text added: "17) PGEC1"
- board text added: "25) GND"
- board text added: "33) RP99/RF3"
- board text added: "48) ACCEL2"
- board text added: "54) Tx"
- board text added: "ACCEL0"
- board text added: "ACCEL1"
- board text added: "AN1/VREF-/RPI33/RB1"
- board text added: "AN8/PMA6/RPI40/RB8"
- board text added: "AN9/PMA7//RPI41/RB9"
- board text added: "ANC0"
- board text added: "ANC1"
- board text added: "ANC2"
- board text added: "CTS"
- board text added: "ENC0"
- board text added: "ENC1"
- board text added: "ENC2"
- board text added: "ENCODER1"
- board text added: "ENCODER2"
- board text added: "ENCODER3"
- board text added: "ENCODER4"
- board text added: "ENCODER5"
- board text added: "ENCODER6"
- board text added: "GND"
- board text added: "GYRO0"
- board text added: "GYRO1"
- board text added: "GYRO2"
- board text added: "LED1"
- board text added: "LED2"
- board text added: "LED3"
- board text added: "LED4"
- board text added: "LED5"
- board text added: "OSC1"
- board text added: "OSC2"
- board text added: "PGED1"
- board text added: "PWM1H (MotorCon1)"
- board text added: "PWM1L (MotorCon0)"
- board text added: "PWM2H (MotorCon3)"
- board text added: "PWM2L (MotorCon2)"
- board text added: "PWM3L (MotorCon4)"
- board text added: "PWM4H (MagnetCon1)"
- board text added: "PWM4L (MagnetCon0)"
- board text added: "RP65/RD1"
- board text added: "RTS"
- board text added: "Rx"
- board text added: "SCL2/PMA8/RP101/RF5"
- board text added: "SDA2/PMA9/RP100/RF4"
- board text added: "SPI_BUS0"
- board text added: "SPI_BUS1"
- board text added: "SPI_BUS2"
- board text added: "TDO/AN11/PMA12/RPI43/RB11"
- board text added: "TMS/AN10/CVREF/PMA13/RPI42/RB10"
- board text added: "VCC"
- board text added: "VCap"
- board text added: "~MCLR"
