File: PCB/DsPIC Breakout/DsPIC Breakout.sch (KiCad schematic (older format))
At the start: 14 parts, among them P1 CONN_2

Commit message: KICad BreakOut Board (64 pin dsPIC)
Schematic and Layout
Parts:
- removed J? (x4): BREADBOARD_HEADER_L, ~, symbol BREADBOARD_HEADER_L
- added CR1: CERAMIC_RES, ~, symbol CERAMIC_RES
- added J1, J2, J3, J4: BREADBOARD_HEADER_16X1, ~, symbol BREADBOARD_HEADER_16X1
- added R2: 1M, ~, symbol R
- C5: renamed from C?; value C -> 0.1uF
- gave numbers to parts that had none: 7
Connections:
- wire segments 214 -> 207
Other:
- moved on the sheet: C3, C5

Commit message: Updated Breakout Board 64pin dsPIC
Parts:
- removed J1, J2, J3, J4: BREADBOARD_HEADER_16X1, ~, symbol BREADBOARD_HEADER_16X1
- added J1, J2: BREADBOARD_HEADER_32X1, ~, symbol BREADBOARD_HEADER_32X1
Connections:
- wire segments 207 -> 278
